File: power.sch (KiCad schematic (older format))
At the start: 31 parts, among them J4 JST_PH, J5 PicoBlade, J6 PicoBlade, Q2 FDC6312P, SW1 Slide Switch, U2 BQ24295, U3 MCP73832-2-MC, U4 MCP1811AT-033/OT

Commit message: almost ready rev a
Parts:
- R12, R13: Variant (none) -> BQ24295
- R6: value 2k -> 1k
Changed lines of the file:
@@
 P 2050 5000
 F 0 "R6" V 1843 5000 50  0000 C CNN
-F 1 "2k" V 1934 5000 50  0000 C CNN
+F 1 "1k" V 1934 5000 50  0000 C CNN
 F 2 "Resistor_SMD:R_0805_2012Metric" V 1980 5000 50  0001 C CNN
 F 3 "~" H 2050 5000 50  0001 C CNN
@@
 F 2 "Resistor_SMD:R_0805_2012Metric" H 1300 4100 50  0001 C CNN
 F 3 "~" H 1300 4100 50  0001 C CNN
+F 4 "BQ24295" H 1300 4100 50  0001 C CNN "Variant"
 	1    1300 4100
 	1    0    0    -1
@@
 F 2 "Resistor_SMD:R_0805_2012Metric" H 1600 4100 50  0001 C CNN
 F 3 "~" H 1600 4100 50  0001 C CNN
+F 4 "BQ24295" H 1600 4100 50  0001 C CNN "Variant"
 	1    1600 4100
 	1    0    0    -1

Commit message: improve power switch circuit
Parts:
- removed F1: 3A, Fuse:Fuseholder_Littelfuse_Nano2_154x, symbol Device:Fuse
- removed J4: JST_PH, Connector_JST:JST_PH_S2B-PH-SM4-TB_1x02-1MP_P2.00mm_Horizontal, symbol Connector_Generic:Conn_01x02
- removed J5: PicoBlade, Connector_Molex:Molex_PicoBlade_53261-0271_1x02-1MP_P1.25mm_Horizontal, symbol Connector_Generic:Conn_01x02
- removed R11: 10k, Resistor_SMD:R_0805_2012Metric, symbol Device:R_Small
- removed SW1: Slide Switch, project:SW_OS102011MS2QN1, symbol Switch:SW_SPDT
- D34: value ~ -> 1N4007; Part (none) -> SOD-123 1N4007
- J6: Variant BQ24295 -> BQ24295,DNP
- TH1: value 10k -> 10k NTC
Connections:
- net PWROFF renamed PWRON
Other:
- note removed: "Battery connector"
- note removed: "Power switch"
- moved on the sheet: C12, C13, R10, U4

Commit message: Rev A complete
Parts:
- LED1: Comment (none) -> 0805
- U2: Part (none) -> BQ24295
- U4: Part MCP1811AT-033/TT -> MCP1811AT-033/OT; PartAlt (none) -> TLV70033DDC
Changed lines of the file:
@@
 $Descr A4 11693 8268
 encoding utf-8
-Sheet 3 3
+Sheet 2 3
 Title ""
 Date ""
@@
 F 3 "https://www.ti.com/lit/ds/symlink/bq24295.pdf" H 2250 3750 50  0001 C CNN
 F 4 "BQ24295" H 2250 2900 50  0001 C CNN "Variant"
+F 5 "BQ24295" H 2250 2900 50  0001 C CNN "Part"
 	1    2250 2900
 	1    0    0    -1
@@
 U 1 1 6083411E
 P 1750 5000
-F 0 "LED1" H 1743 4745 50  0000 C CNN
-F 1 "Red" H 1743 4836 50  0000 C CNN
+F 0 "LED1" H 1743 4655 50  0000 C CNN
+F 1 "Red" H 1743 4746 50  0000 C CNN
 F 2 "LED_SMD:LED_0805_2012Metric" H 1750 5000 50  0001 C CNN
 F 3 "~" H 1750 5000 50  0001 C CNN
+F 4 "0805" H 1743 4837 50  0000 C CNN "Comment"
 	1    1750 5000
 	-1   0    0    1
@@
 F 2 "Package_TO_SOT_SMD:SOT-23-5" H 9500 2200 50  0001 C CNN
 F 3 "http://ww1.microchip.com/downloads/en/DeviceDoc/MCP1811A-11B-12A-12B-Data-Sheet-20006088B.pdf" H 9500 2000 50  0001 C CNN
-F 4 "MCP1811AT-033/TT" H 9500 2000 50  0001 C CNN "Part"
+F 4 "MCP1811AT-033/OT" H 9500 2000 50  0001 C CNN "Part"
+F 5 "TLV70033DDC" H 9500 2000 50  0001 C CNN "PartAlt"
 	1    9500 2000
 	1    0    0    -1
