File: power.sch (KiCad schematic (older format))
At the start: 26 parts, among them J6 PicoBlade, Q2 FDC6312P, U2 BQ24295, U3 MCP73832-2-MC, U4 MCP1811AT-033/OT

Commit message: archive footprints and schematics symbols
Parts:
- C10, C11, C12, C13, C5, C7, C8: footprint Capacitor_SMD:C_0805_2012Metric -> archive:C_0805_2012Metric; symbol Device:C_Small -> archive:Device_C_Small
- C6, C9: footprint Capacitor_SMD:C_1206_3216Metric -> archive:C_1206_3216Metric; symbol Device:C_Small -> archive:Device_C_Small
- D34: footprint Diode_SMD:D_SOD-123 -> archive:D_SOD-123; symbol Device:D -> archive:Device_D
- J6: footprint Connector_Molex:Molex_PicoBlade_53261-0271_1x02-1MP_P1.25mm_Horizontal -> archive:Molex_PicoBlade_53261-0271_1x02-1MP_P1.25mm_Horizontal; symbol Connector_Generic:Conn_01x02 -> archive:Connector_Generic_Conn_01x02
- JP100: footprint project:GND_Tie -> archive:GND_Tie; symbol Jumper:SolderJumper_2_Bridged -> archive:Jumper_SolderJumper_2_Bridged
- L1: footprint Inductor_SMD:L_Bourns-SRN4018 -> archive:L_Bourns-SRN4018; symbol Device:L -> archive:Device_L
- LED1: footprint LED_SMD:LED_0805_2012Metric -> archive:LED_0805_2012Metric; symbol Device:LED -> archive:Device_LED
- Q2: footprint Package_TO_SOT_SMD:SuperSOT-6 -> archive:SuperSOT-6; symbol Device:Q_Dual_PMOS_G1S2G2D2S1D1 -> archive:Device_Q_Dual_PMOS_G1S2G2D2S1D1
- R10, R12, R13, R7, R8: footprint Resistor_SMD:R_0805_2012Metric -> archive:R_0805_2012Metric; symbol Device:R_Small -> archive:Device_R_Small
- R6, R9: footprint Resistor_SMD:R_0805_2012Metric -> archive:R_0805_2012Metric; symbol Device:R -> archive:Device_R
- TH1: footprint Resistor_SMD:R_0805_2012Metric -> archive:R_0805_2012Metric; symbol Device:Thermistor_NTC -> archive:Device_Thermistor_NTC
- U2: footprint Package_DFN_QFN:QFN-24-1EP_4x4mm_P0.5mm_EP2.65x2.65mm -> archive:QFN-24-1EP_4x4mm_P0.5mm_EP2.65x2.65mm; symbol project:BQ24295 -> archive:project_BQ24295
- U3: footprint Package_DFN_QFN:DFN-8-1EP_3x2mm_P0.5mm_EP1.7x1.4mm -> archive:DFN-8-1EP_3x2mm_P0.5mm_EP1.7x1.4mm; symbol project:MCP73832-2-MC -> archive:project_MCP73832-2-MC
- U4: footprint Package_TO_SOT_SMD:SOT-23-5 -> archive:SOT-23-5; symbol project:MCP1811 -> archive:project_MCP1811
