File: keyboard.sch (KiCad schematic (older format))
At the start: 22 parts, among them J1 Conn_SWD, J2 Conn_ETM, J3 USB_C_Receptacle, J7 2.54mm, J8 PicoBlade, J9 PicoBlade, Q1 IRLML2502, U1 BL653, Y1 32.768kHz

Commit message: all routed
Connections:
- no-connect marks 12 -> 17
Changed lines of the file:
@@
 	1    0    0    -1
 $EndComp
+NoConn ~ 4100 3000
+NoConn ~ 4100 2900
+NoConn ~ 4100 2800
+NoConn ~ 4100 2600
+NoConn ~ 4100 2400
+Wire Wire Line
+	4100 2400 3700 2400
+Wire Wire Line
+	4100 2800 3700 2800
+Wire Wire Line
+	4100 2600 3700 2600
+Wire Wire Line
+	4100 2900 3700 2900
 Wire Bus Line
 	1800 4300 1800 4800

Commit message: improve power switch circuit
Parts:
- added C16: 1uF, Capacitor_SMD:C_0805_2012Metric, symbol Device:C_Small
- added D35, D36: 1N4007, Diode_SMD:D_SOD-123, symbol Device:D_Small
- added F1: 3A, Fuse:Fuseholder_Littelfuse_Nano2_154x, symbol Device:Fuse
- added J4: JST_PH, Connector_JST:JST_PH_S2B-PH-SM4-TB_1x02-1MP_P2.00mm_Horizontal, symbol Connector_Generic:Conn_01x02
- added J5: PicoBlade, Connector_Molex:Molex_PicoBlade_53261-0271_1x02-1MP_P1.25mm_Horizontal, symbol Connector_Generic:Conn_01x02
- added R11: 10k, Resistor_SMD:R_0805_2012Metric, symbol Device:R_Small
- added R15, R16: 100k, Resistor_SMD:R_0805_2012Metric, symbol Device:R_Small
- added SW1: Slide Switch, project:SW_OS102011MS2QN1, symbol Switch:SW_SPDT
- Q1: value IRLML2502 -> 2N7002; Part IRLML2502 -> 2N7002
Connections:
- net GND: now also C16.2, R16.1
- net VBAT: now also F1.1
- net VBUS: now also R11.1
- new net: F1.2, J4.1 (Pin_1), J5.1 (Pin_1)
- new net: D35.1 (K), SW1.1 (A)
- new net: R16.2, SW1.3 (C)
- new net: D36.2 (A), R11.2
- new net: D35.2 (A), R15.2
- new net GNDPWR: J4.2 (Pin_2), J5.2 (Pin_2)
- new net PWRON: C16.1, D36.1 (K), SW1.2 (B)
- new net VSYS: R15.1
Other:
- note added: "100ms switch debounce"
- note added: "Battery connector"
- note added: "Choice of 2 battery connectors"
- note added: "Debug & expansion connectors"
- note added: "Force power on when 5V connected\nto allow mcu to configure charger"
- note added: "Off"
- note added: "On"
- note added: "Power switch"
- note removed: "Debug Connectors"

Commit message: final changes to power switch circuitry
Parts:
- removed R11: 10k, Resistor_SMD:R_0805_2012Metric, symbol Device:R_Small
- R15, R16: value 100k -> 10k
Connections:
- net VBUS: now also D36.2 (A)
Other:
- note added: "10ms switch debounce"
- note added: "Battery\nvoltage\nsense\ndivider"
- note removed: "100ms switch debounce"
- moved on the sheet: C16, D35, D36, LED2, R14, R15, R16, SW1

Commit message: Rev A complete
Parts:
- added LED3: Red, LED_THT:LED_D3.0mm, symbol Device:LED
- LED2: symbol Device:LED_Small -> Device:LED; Comment (none) -> 0805
- Y1: Comment CL=9pf -> CL=12.5pf
Connections:
- net +3V3: now also LED3.2 (A)
- net at LED2.1 (K), R14.1: now also LED3.1 (K)
Other:
- note added: "Choice of smd and tht\nfor caps lock led"
- moved on the sheet: C16, D35, D36, F1, J4, J5, LED2, R14, R15, R16, SW1
