File: matrix.sch (KiCad schematic (older format))
At the start: 97 parts

Commit message: almost ready rev a
Parts:
- D1, D10, D11, D12, D13, D14, D15, D16, D17, D18, D19, D2, D20, D21, D22, D23, D24, D25, D26, D27, D28, D29, D3, D30, D31, D32, D33, D4, D5, D6, D7, D8, D9: value D_Dual_CommonAnode_KKA_Split -> BAS70-06

Commit message: Rev A complete
Parts:
- S1, S10, S11, S12, S13, S14, S15, S16, S17, S18, S19, S2, S20, S21, S22, S23, S24, S25, S26, S27, S28, S29, S3, S30, S31, S32, S33, S34, S35, S36, S37, S38, S39, S4, S40, S41, S42, S43, S44, S45, S46, S47, S48, S49, S5, S50, S51, S52, S53, S54, S55, S56, S57, S58, S59, S6, S60, S61, S62, S63, S64, S7, S8, S9: value SW_Push -> MX1A

Commit message: Change diode part BAS70 -> BAT54
Use lower voltage diode for better forward voltage
Parts:
- D1, D10, D11, D12, D13, D14, D15, D16, D17, D18, D19, D2, D20, D21, D22, D23, D24, D25, D26, D27, D28, D29, D3, D30, D31, D32, D33, D4, D5, D6, D7, D8, D9: value BAS70-06 -> BAT54A; Part BAS70-06 -> BAT54A

Commit message: archive footprints and schematics symbols
Parts:
- D1, D10, D11, D12, D13, D14, D15, D16, D17, D18, D19, D2, D20, D21, D22, D23, D24, D25, D26, D27, D28, D29, D3, D30, D31, D32, D33, D4, D5, D6, D7, D8, D9: footprint Package_TO_SOT_SMD:SOT-23 -> archive:SOT-23; symbol Device:D_Dual_CommonAnode_KKA_Split -> archive:Device_D_Dual_CommonAnode_KKA_Split
- S1, S10, S11, S12, S13, S16, S17, S18, S19, S2, S20, S21, S22, S23, S24, S25, S26, S27, S3, S30, S31, S32, S33, S34, S35, S36, S37, S38, S39, S4, S40, S43, S44, S45, S46, S47, S48, S49, S5, S50, S51, S52, S53, S54, S55, S6, S60, S61, S62, S63, S64, S7, S8, S9: footprint Button_Switch_Keyboard:SW_Cherry_MX_1.00u_PCB -> archive:SW_Cherry_MX_1.00u_PCB; symbol Switch:SW_Push -> archive:Switch_SW_Push
- S14, S42: footprint Button_Switch_Keyboard:SW_Cherry_MX_2.00u_PCB -> archive:SW_Cherry_MX_2.00u_PCB; symbol Switch:SW_Push -> archive:Switch_SW_Push
- S15, S28: footprint Button_Switch_Keyboard:SW_Cherry_MX_1.50u_PCB -> archive:SW_Cherry_MX_1.50u_PCB; symbol Switch:SW_Push -> archive:Switch_SW_Push
- S29: footprint Button_Switch_Keyboard:SW_Cherry_MX_1.75u_PCB -> archive:SW_Cherry_MX_1.75u_PCB; symbol Switch:SW_Push -> archive:Switch_SW_Push
- S41: footprint Button_Switch_Keyboard:SW_Cherry_MX_2.25u_PCB -> archive:SW_Cherry_MX_2.25u_PCB; symbol Switch:SW_Push -> archive:Switch_SW_Push
- S56, S57, S58: footprint Button_Switch_Keyboard:SW_Cherry_MX_1.25u_PCB -> archive:SW_Cherry_MX_1.25u_PCB; symbol Switch:SW_Push -> archive:Switch_SW_Push
- S59: footprint Button_Switch_Keyboard:SW_Cherry_MX_6.25u_PCB -> archive:SW_Cherry_MX_6.25u_PCB; symbol Switch:SW_Push -> archive:Switch_SW_Push
